File: Intro Board v1/Intro Board v1.kicad_pcb (KiCad board)
At the start: 4 copper layers, 75 x 25 mm, 63 parts, among them J1 3220-20-0200-00, J2 GSB1C41110SSHR, J3 1984617, J4 647676-2, Q1 NMOS, U1 LMS8117AMP-3.3_NOPB, U2 SST25VF010A-33-4C-SAE, U4 BMP390, U5 CP2102N-A02-GQFN20, U7 STM32G441KBT6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

Commit message: PATRICK BOARD V2
Routing:
- net GND: track 88.7 -> 97.9 mm, vias 30 -> 41
- net +3.3V: track 64.1 -> 66.8 mm, vias 16 -> 18

Commit message: PATRICK BOARD V3
Routing:
- net +3.3V: track 66.8 -> 69.1 mm, vias 18 -> 20
